File: hardware/PCB/TRACE_PCB.kicad_sch (KiCad schematic)
At the start: 0 parts

Commit message: Completed schematic
Parts:
- added H1, H2, H3, H4: MountingHole, MountingHole:MountingHole_3.2mm_M3, symbol Mechanical:MountingHole
- added J17: DigitalPower, Connector_PinHeader_2.54mm:PinHeader_1x03_P2.54mm_Vertical, symbol Connector:Conn_01x03_Pin
- added J18: AnalogPower, Connector_PinHeader_2.54mm:PinHeader_1x02_P2.54mm_Vertical, symbol Connector:Conn_01x02_Pin
- added J19: SymetricPower, Connector_PinHeader_2.54mm:PinHeader_1x02_P2.54mm_Vertical, symbol Connector:Conn_01x02_Pin
Connections:
- new net +12V: J19.1 (Pin_1)
- new net +3.3V: J17.2 (Pin_2)
- new net +3.3VA: J18.1 (Pin_1)
- new net +5V: J17.1 (Pin_1)
- new net -12V: J19.2 (Pin_2)
- new net GND: J17.3 (Pin_3)
- new net GNDA: J18.2 (Pin_2)
Other:
- sheet ESP32S3 ports: added RXD0, TXD0; removed none
- sheet RP2350Schematic ports: added RP_RXD0, RP_TXD0, triggerOut; removed none
- sheet Scope ports: added triggerOut; removed none
