File: hardware/PCB/esp32s3.kicad_sch (KiCad schematic)
At the start: 42 parts, among them J5 ISP_Programmer, P1 USB_C_Plug, Q1 PMOS, Q2 PMOS, Q3 PMOS, Q4 PMOS, Q5 NMOS, Q6 NMOS, Q7 PMOS, Q8 PMOS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

Commit message: Completed schematic
Parts:
- added C92, C93: 100nF, Capacitor_SMD:C_0603_1608Metric_Pad1.08x0.95mm_HandSolder, symbol Device:C_Small
- added C96: 220uF, Capacitor_SMD:CP_Elec_6.3x5.3, symbol Device:C_Polarized_Small
- added D5, D6: WS2812B, LED_SMD:LED_WS2812B_PLCC4_5.0x5.0mm_P3.2mm, symbol LED:WS2812B
- added J11: Internal I²C, Connector_PinHeader_2.54mm:PinHeader_1x04_P2.54mm_Vertical, symbol Connector:Conn_01x04_Pin
- added J12: External I²C, Connector_PinHeader_2.54mm:PinHeader_1x04_P2.54mm_Horizontal, symbol Connector:Conn_01x04_Pin
- added J13: External SPI, Connector_PinHeader_2.54mm:PinHeader_1x06_P2.54mm_Horizontal, symbol Connector:Conn_01x06_Pin
- added J14: External UART, Connector_PinHeader_2.54mm:PinHeader_1x04_P2.54mm_Horizontal, symbol Connector:Conn_01x04_Pin
- added J15: Internal UART, Connector_PinHeader_2.54mm:PinHeader_1x04_P2.54mm_Vertical, symbol Connector:Conn_01x04_Pin
- added J16: Internal SPI, Connector_PinHeader_2.54mm:PinHeader_1x05_P2.54mm_Vertical, symbol Connector:Conn_01x05_Pin
- added R67, R68: 4.7kΩ, Resistor_SMD:R_0603_1608Metric_Pad0.98x0.95mm_HandSolder, symbol Device:R_Small
- added R70: 100Ω, Resistor_SMD:R_0603_1608Metric_Pad0.98x0.95mm_HandSolder, symbol Device:R_Small
Connections:
- net +3.3V: now also C96.1, J11.3 (Pin_3), J12.3 (Pin_3), J13.5 (Pin_5), J14.3 (Pin_3), J15.3 (Pin_3), J16.4 (Pin_4), R67.1, R68.1
- net +5V: now also C92.2, C93.2, D5.1 (VDD), D6.1 (VDD)
- net GND: now also C92.1, C93.1, C96.2, D5.3 (VSS), D6.3 (VSS), J11.4 (Pin_4), J12.4 (Pin_4), J13.6 (Pin_6), J14.4 (Pin_4), J15.4 (Pin_4), J16.5 (Pin_5)
- net MISO: now also J16.3 (Pin_3)
- net MOSI: now also J16.2 (Pin_2)
- net RXD0: now also J15.2 (Pin_2)
- net SCK: now also J16.1 (Pin_1)
- net SCL: now also J11.1 (Pin_1)
- net SDA: now also J11.2 (Pin_2)
- net TXD0: now also J15.1 (Pin_1)
- net IO1 renamed E_SDA
- net E_SDA: now also J12.1 (Pin_1), R68.2
- net IO2 renamed E_SCL
- net E_SCL: now also J12.2 (Pin_2), R67.2
- net IO3 renamed E_CS
- net E_CS: now also J13.1 (Pin_1)
- net IO39 renamed E_TX
- net E_TX: now also J14.1 (Pin_1)
- net IO4 renamed E_SCK
- net E_SCK: now also J13.2 (Pin_2)
- net IO40 renamed E_RX
- net E_RX: now also J14.2 (Pin_2)
- net IO41 renamed RGB_LED
- net RGB_LED: now also R70.2
- net IO5 renamed E_MISO
- net E_MISO: now also J13.3 (Pin_3)
- net IO6 renamed E_MOSI
- net E_MOSI: now also J13.4 (Pin_4)
- new net: D5.2 (DOUT), D6.4 (DIN)
- new net: D5.4 (DIN), R70.1
- no-connect marks 15 -> 16
Other:
- note added: "Connectors"
- note added: "WS2812B status LEDs"
