File: hardware/PCB/rp2350Schematic.kicad_sch (KiCad schematic)
At the start: 62 parts, among them J6 LogicAnalyzerHeader, J7 SWDHeader, J8 SWD_Programmer, P2 USB_C_Plug, SW3 Reset, SW4 Run, U14 RP2350B-QFN80, U15 W25Q128JVS, U16 SN74LVC245APW, U17 AMS1117-3.3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

Commit message: Completed schematic
Parts:
- added C91: 220uF, Capacitor_SMD:CP_Elec_6.3x5.3, symbol Device:C_Polarized_Small
- added C94, C95: 100nF, Capacitor_SMD:C_0603_1608Metric_Pad1.08x0.95mm_HandSolder, symbol Device:C_Small
- added D7, D8: WS2812B, LED_SMD:LED_WS2812B_PLCC4_5.0x5.0mm_P3.2mm, symbol LED:WS2812B
- added R71: 100Ω, Resistor_SMD:R_0603_1608Metric_Pad0.98x0.95mm_HandSolder, symbol Device:R_Small
Connections:
- net +3.3VP: now also C91.1
- net +5V: now also C94.2, C95.2, D7.1 (VDD), D8.1 (VDD)
- net GND: now also C91.2, C94.1, C95.1, D7.3 (VSS), D8.3 (VSS)
- net LA_DIR: now reaches R64.2, U14.6 (GPIO8), U16.1 (DIR)
- net LA_~{OE}: now reaches R57.2, U14.7 (GPIO9), U16.19 (~{OE})
- net RP_TXD0: now reaches U14.36 (GPIO28)
- net RP_RXD0: now reaches U14.37 (GPIO29)
- net RGB_LED: now reaches U14.38 (GPIO30)
- net RGB_LED: now also R71.2
- net triggerOut: now reaches U14.39 (GPIO31)
- new net: D7.4 (DIN), D8.2 (DOUT)
- new net: D8.4 (DIN), R71.1
- no-connect marks 11 -> 12
Other:
- note added: "3.3V voltage source"
- note added: "Logic Anaylzer"
- note added: "MCU with flash"
- note added: "Ws2812B status LEDs"
- moved on the sheet: C62, C63, C64, C65, C66, C67, C68, C69, C70, C74, C77, C78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
